Commit message: Expand the functionality, for multiple drives (#8)
* Expand the functionality, for multiple drives

* Update URDF etc. for 2 joints

* README updates

File: description/ros2_control/two_dof.ros2_control.xacro (robot description, xacro)
@@ -1,10 +1,8 @@
 <?xml version="1.0"?>
 <robot xmlns:xacro="http://www.ros.org/wiki/xacro">
-  <xacro:macro name="single_dof_ros2_control" params="name prefix">
+  <xacro:macro name="two_dof_ros2_control" params="name prefix">
     <ros2_control name="${name}" type="system">
       <hardware>
         <plugin>synapticon_ros2_control/SynapticonSystemInterface</plugin>
-        <!-- For testing, GenericSystem is much simpler and doesn't depend on the code in this package -->
-        <!-- plugin>mock_components/GenericSystem</plugin -->
         <param name="interface_name">eno0</param>
       </hardware>
@@ -19,4 +17,14 @@
         <state_interface name="effort"/>
       </joint>
+      <joint name="${prefix}joint2">
+        <command_interface name="position"/>
+        <command_interface name="velocity"/>
+        <command_interface name="effort"/>
+        <command_interface name="quick_stop"/>
+        <state_interface name="position"/>
+        <state_interface name="velocity"/>
+        <state_interface name="acceleration"/>
+        <state_interface name="effort"/>
+      </joint>
     </ros2_control>
   </xacro:macro>
