Commit message: fix interface_name parsing via argument for single_dof and two_dof

File: description/ros2_control/single_dof.ros2_control.xacro (robot description, xacro)
@@ -1,11 +1,8 @@
 <?xml version="1.0"?>
 <robot xmlns:xacro="http://www.ros.org/wiki/xacro">
-  <xacro:arg name="interface_name" default="eno0"/>
-  <xacro:macro name="single_dof_ros2_control" params="name prefix">
+  <xacro:macro name="single_dof_ros2_control" params="name prefix interface_name">
     <ros2_control name="${name}" type="system">
       <hardware>
         <plugin>synapticon_ros2_control/SynapticonSystemInterface</plugin>
-        <!-- For testing, GenericSystem is much simpler and doesn't depend on the code in this package -->
-        <!-- plugin>mock_components/GenericSystem</plugin -->
         <param name="interface_name">${interface_name}</param>
       </hardware>

File: description/ros2_control/two_dof.ros2_control.xacro (robot description, xacro)
@@ -1,6 +1,5 @@
 <?xml version="1.0"?>
 <robot xmlns:xacro="http://www.ros.org/wiki/xacro">
-  <xacro:arg name="interface_name" default="eno0"/>
-  <xacro:macro name="two_dof_ros2_control" params="name prefix">
+  <xacro:macro name="two_dof_ros2_control" params="name prefix interface_name">
     <ros2_control name="${name}" type="system">
       <hardware>

File: description/urdf/single_dof_in_world.urdf.xacro (robot description, xacro)
@@ -2,4 +2,5 @@
 <robot xmlns:xacro="http://www.ros.org/wiki/xacro" name="single_dof">
   <xacro:arg name="prefix" default="" />
+  <xacro:arg name="interface_name" default="" />
   <xacro:include filename="$(find synapticon_ros2_control)/urdf/single_dof_macro.urdf.xacro" />
   <xacro:include filename="$(find synapticon_ros2_control)/ros2_control/single_dof.ros2_control.xacro" />
@@ -8,4 +9,4 @@
     <origin xyz="0 0 0" rpy="0 0 0" />
   </xacro:single_dof>
-  <xacro:single_dof_ros2_control name="SingleDofRos2Control" prefix="$(arg prefix)" />
+  <xacro:single_dof_ros2_control name="SingleDofRos2Control" prefix="$(arg prefix)" interface_name="$(arg interface_name)" />
 </robot>

File: description/urdf/two_dof_in_world.urdf.xacro (robot description, xacro)
@@ -2,4 +2,5 @@
 <robot xmlns:xacro="http://www.ros.org/wiki/xacro" name="two_dof">
   <xacro:arg name="prefix" default="" />
+  <xacro:arg name="interface_name" default="" />
   <xacro:include filename="$(find synapticon_ros2_control)/urdf/two_dof_macro.urdf.xacro" />
   <xacro:include filename="$(find synapticon_ros2_control)/ros2_control/two_dof.ros2_control.xacro" />
@@ -8,4 +9,4 @@
     <origin xyz="0 0 0" rpy="0 0 0" />
   </xacro:two_dof>
-  <xacro:two_dof_ros2_control name="TwoDofRos2Control" prefix="$(arg prefix)" />
+  <xacro:two_dof_ros2_control name="TwoDofRos2Control" prefix="$(arg prefix)" interface_name="$(arg interface_name)" />
 </robot>

Commit message: rename interface_name to eth_device to prevent name collission with ros2_control interface_name (position, velocity etc)

File: description/ros2_control/single_dof.ros2_control.xacro (robot description, xacro)
@@ -1,9 +1,9 @@
 <?xml version="1.0"?>
 <robot xmlns:xacro="http://www.ros.org/wiki/xacro">
-  <xacro:macro name="single_dof_ros2_control" params="name prefix interface_name">
+  <xacro:macro name="single_dof_ros2_control" params="name prefix eth_device">
     <ros2_control name="${name}" type="system">
       <hardware>
         <plugin>synapticon_ros2_control/SynapticonSystemInterface</plugin>
-        <param name="interface_name">${interface_name}</param>
+        <param name="eth_device">${eth_device}</param>
       </hardware>
       <joint name="${prefix}joint1">

File: description/ros2_control/two_dof.ros2_control.xacro (robot description, xacro)
@@ -1,9 +1,9 @@
 <?xml version="1.0"?>
 <robot xmlns:xacro="http://www.ros.org/wiki/xacro">
-  <xacro:macro name="two_dof_ros2_control" params="name prefix interface_name">
+  <xacro:macro name="two_dof_ros2_control" params="name prefix eth_device">
     <ros2_control name="${name}" type="system">
       <hardware>
         <plugin>synapticon_ros2_control/SynapticonSystemInterface</plugin>
-        <param name="interface_name">${interface_name}</param>
+        <param name="eth_device">${eth_device}</param>
       </hardware>
       <joint name="${prefix}joint1">

File: description/urdf/single_dof_in_world.urdf.xacro (robot description, xacro)
@@ -2,5 +2,5 @@
 <robot xmlns:xacro="http://www.ros.org/wiki/xacro" name="single_dof">
   <xacro:arg name="prefix" default="" />
-  <xacro:arg name="interface_name" default="" />
+  <xacro:arg name="eth_device" default="" />
   <xacro:include filename="$(find synapticon_ros2_control)/urdf/single_dof_macro.urdf.xacro" />
   <xacro:include filename="$(find synapticon_ros2_control)/ros2_control/single_dof.ros2_control.xacro" />
@@ -9,4 +9,4 @@
     <origin xyz="0 0 0" rpy="0 0 0" />
   </xacro:single_dof>
-  <xacro:single_dof_ros2_control name="SingleDofRos2Control" prefix="$(arg prefix)" interface_name="$(arg interface_name)" />
+  <xacro:single_dof_ros2_control name="SingleDofRos2Control" prefix="$(arg prefix)" eth_device="$(arg eth_device)" />
 </robot>

File: description/urdf/two_dof_in_world.urdf.xacro (robot description, xacro)
@@ -2,5 +2,5 @@
 <robot xmlns:xacro="http://www.ros.org/wiki/xacro" name="two_dof">
   <xacro:arg name="prefix" default="" />
-  <xacro:arg name="interface_name" default="" />
+  <xacro:arg name="eth_device" default="" />
   <xacro:include filename="$(find synapticon_ros2_control)/urdf/two_dof_macro.urdf.xacro" />
   <xacro:include filename="$(find synapticon_ros2_control)/ros2_control/two_dof.ros2_control.xacro" />
@@ -9,4 +9,4 @@
     <origin xyz="0 0 0" rpy="0 0 0" />
   </xacro:two_dof>
-  <xacro:two_dof_ros2_control name="TwoDofRos2Control" prefix="$(arg prefix)" interface_name="$(arg interface_name)" />
+  <xacro:two_dof_ros2_control name="TwoDofRos2Control" prefix="$(arg prefix)" eth_device="$(arg eth_device)" />
 </robot>

Commit message: Add mechanical reduction parameters

File: description/ros2_control/single_dof.ros2_control.xacro (robot description, xacro)
@@ -1,9 +1,10 @@
 <?xml version="1.0"?>
 <robot xmlns:xacro="http://www.ros.org/wiki/xacro">
-  <xacro:macro name="single_dof_ros2_control" params="name prefix eth_device">
+  <xacro:macro name="single_dof_ros2_control" params="name prefix eth_device joint1_mechanical_reduction">
     <ros2_control name="${name}" type="system">
       <hardware>
         <plugin>synapticon_ros2_control/SynapticonSystemInterface</plugin>
         <param name="eth_device">${eth_device}</param>
+        <param name="joint1_mechanical_reduction">${joint1_mechanical_reduction}</param>
       </hardware>
       <joint name="${prefix}joint1">

File: description/ros2_control/two_dof.ros2_control.xacro (robot description, xacro)
@@ -1,9 +1,11 @@
 <?xml version="1.0"?>
 <robot xmlns:xacro="http://www.ros.org/wiki/xacro">
-  <xacro:macro name="two_dof_ros2_control" params="name prefix eth_device">
+  <xacro:macro name="two_dof_ros2_control" params="name prefix eth_device joint1_mechanical_reduction joint2_mechanical_reduction">
     <ros2_control name="${name}" type="system">
       <hardware>
         <plugin>synapticon_ros2_control/SynapticonSystemInterface</plugin>
         <param name="eth_device">${eth_device}</param>
+        <param name="joint1_mechanical_reduction">${joint1_mechanical_reduction}</param>
+        <param name="joint2_mechanical_reduction">${joint2_mechanical_reduction}</param>
       </hardware>
       <joint name="${prefix}joint1">

File: description/urdf/single_dof_in_world.urdf.xacro (robot description, xacro)
@@ -3,4 +3,5 @@
   <xacro:arg name="prefix" default="" />
   <xacro:arg name="eth_device" default="" />
+  <xacro:arg name="joint1_mechanical_reduction" default="1.0" />
   <xacro:include filename="$(find synapticon_ros2_control)/urdf/single_dof_macro.urdf.xacro" />
   <xacro:include filename="$(find synapticon_ros2_control)/ros2_control/single_dof.ros2_control.xacro" />
@@ -9,4 +10,4 @@
     <origin xyz="0 0 0" rpy="0 0 0" />
   </xacro:single_dof>
-  <xacro:single_dof_ros2_control name="SingleDofRos2Control" prefix="$(arg prefix)" eth_device="$(arg eth_device)" />
+  <xacro:single_dof_ros2_control name="SingleDofRos2Control" prefix="$(arg prefix)" eth_device="$(arg eth_device)" joint1_mechanical_reduction="$(arg joint1_mechanical_reduction)" />
 </robot>

File: description/urdf/two_dof_in_world.urdf.xacro (robot description, xacro)
@@ -3,4 +3,6 @@
   <xacro:arg name="prefix" default="" />
   <xacro:arg name="eth_device" default="" />
+  <xacro:arg name="joint1_mechanical_reduction" default="1.0" />
+  <xacro:arg name="joint2_mechanical_reduction" default="1.0" />
   <xacro:include filename="$(find synapticon_ros2_control)/urdf/two_dof_macro.urdf.xacro" />
   <xacro:include filename="$(find synapticon_ros2_control)/ros2_control/two_dof.ros2_control.xacro" />
@@ -9,4 +11,4 @@
     <origin xyz="0 0 0" rpy="0 0 0" />
   </xacro:two_dof>
-  <xacro:two_dof_ros2_control name="TwoDofRos2Control" prefix="$(arg prefix)" eth_device="$(arg eth_device)" />
+  <xacro:two_dof_ros2_control name="TwoDofRos2Control" prefix="$(arg prefix)" eth_device="$(arg eth_device)" joint1_mechanical_reduction="$(arg joint1_mechanical_reduction)" joint2_mechanical_reduction="$(arg joint2_mechanical_reduction)"/>
 </robot>
