Commit message: Update joint names to match ROBIN for 7-dof case (#30)
* Update joint names to match ROBIN for 7-dof case

* Fix mechanical reduction param passing

File: description/ros2_control/seven_dof.ros2_control.xacro (robot description, xacro)
@@ -3,19 +3,19 @@
   <xacro:macro name="seven_dof_ros2_control" params="name
     prefix eth_device
-    joint1_mechanical_reduction joint2_mechanical_reduction joint3_mechanical_reduction joint4_mechanical_reduction
-    joint5_mechanical_reduction joint6_mechanical_reduction joint7_mechanical_reduction">
+    yaw1_mechanical_reduction yaw2_mechanical_reduction elev1_j1_mechanical_reduction elev1_j2_mechanical_reduction
+    wrist_yaw_mechanical_reduction wrist_pitch_mechanical_reduction wrist_roll_mechanical_reduction">
     <ros2_control name="${name}" type="system">
       <hardware>
         <plugin>synapticon_ros2_control/SynapticonSystemInterface</plugin>
         <param name="eth_device">${eth_device}</param>
-        <param name="joint1_mechanical_reduction">${joint1_mechanical_reduction}</param>
-        <param name="joint2_mechanical_reduction">${joint2_mechanical_reduction}</param>
-        <param name="joint3_mechanical_reduction">${joint3_mechanical_reduction}</param>
-        <param name="joint4_mechanical_reduction">${joint4_mechanical_reduction}</param>
-        <param name="joint5_mechanical_reduction">${joint5_mechanical_reduction}</param>
-        <param name="joint6_mechanical_reduction">${joint6_mechanical_reduction}</param>
-        <param name="joint7_mechanical_reduction">${joint7_mechanical_reduction}</param>
+        <param name="yaw1_mechanical_reduction">${yaw1_mechanical_reduction}</param>
+        <param name="yaw2_mechanical_reduction">${yaw2_mechanical_reduction}</param>
+        <param name="elev1_j1_mechanical_reduction">${elev1_j1_mechanical_reduction}</param>
+        <param name="elev1_j2_mechanical_reduction">${elev1_j2_mechanical_reduction}</param>
+        <param name="wrist_yaw_mechanical_reduction">${wrist_yaw_mechanical_reduction}</param>
+        <param name="wrist_pitch_mechanical_reduction">${wrist_pitch_mechanical_reduction}</param>
+        <param name="wrist_roll_mechanical_reduction">${wrist_roll_mechanical_reduction}</param>
       </hardware>
-      <joint name="${prefix}joint1">
+      <joint name="${prefix}yaw1">
         <command_interface name="position"/>
         <command_interface name="velocity"/>
@@ -30,5 +30,5 @@
         <state_interface name="hand_guided"/>
       </joint>
-      <joint name="${prefix}joint2">
+      <joint name="${prefix}yaw2">
         <command_interface name="position"/>
         <command_interface name="velocity"/>
@@ -43,5 +43,5 @@
         <state_interface name="hand_guided"/>
       </joint>
-      <joint name="${prefix}joint3">
+      <joint name="${prefix}elev1_j1">
         <command_interface name="position"/>
         <command_interface name="velocity"/>
@@ -56,5 +56,5 @@
         <state_interface name="hand_guided"/>
       </joint>
-      <joint name="${prefix}joint4">
+      <joint name="${prefix}elev1_j2">
         <command_interface name="position"/>
         <command_interface name="velocity"/>
@@ -69,5 +69,5 @@
         <state_interface name="hand_guided"/>
       </joint>
-      <joint name="${prefix}joint5">
+      <joint name="${prefix}wrist_yaw">
         <command_interface name="position"/>
         <command_interface name="velocity"/>
@@ -82,5 +82,5 @@
         <state_interface name="hand_guided"/>
       </joint>
-      <joint name="${prefix}joint6">
+      <joint name="${prefix}wrist_pitch">
         <command_interface name="position"/>
         <command_interface name="velocity"/>
@@ -95,5 +95,5 @@
         <state_interface name="hand_guided"/>
       </joint>
-      <joint name="${prefix}joint7">
+      <joint name="${prefix}wrist_roll">
         <command_interface name="position"/>
         <command_interface name="velocity"/>

File: description/urdf/seven_dof_in_world.urdf.xacro (robot description, xacro)
@@ -3,11 +3,11 @@
   <xacro:arg name="prefix" default="" />
   <xacro:arg name="eth_device" default="" />
-  <xacro:arg name="joint1_mechanical_reduction" default="169.85" />
-  <xacro:arg name="joint2_mechanical_reduction" default="169.85" />
-  <xacro:arg name="joint3_mechanical_reduction" default="1.0" />
-  <xacro:arg name="joint4_mechanical_reduction" default="169.85" />
-  <xacro:arg name="joint5_mechanical_reduction" default="169.85" />
-  <xacro:arg name="joint6_mechanical_reduction" default="169.85" />
-  <xacro:arg name="joint7_mechanical_reduction" default="169.85" />
+  <xacro:arg name="yaw1_mechanical_reduction" default="169.85" />
+  <xacro:arg name="yaw2_mechanical_reduction" default="169.85" />
+  <xacro:arg name="elev1_j1_mechanical_reduction" default="1.0" />
+  <xacro:arg name="elev1_j2_mechanical_reduction" default="169.85" />
+  <xacro:arg name="wrist_yaw_mechanical_reduction" default="169.85" />
+  <xacro:arg name="wrist_pitch_mechanical_reduction" default="169.85" />
+  <xacro:arg name="wrist_roll_mechanical_reduction" default="169.85" />
   <xacro:include filename="$(find synapticon_ros2_control)/urdf/seven_dof_macro.urdf.xacro" />
   <xacro:include filename="$(find synapticon_ros2_control)/ros2_control/seven_dof.ros2_control.xacro" />
@@ -19,10 +19,10 @@
     prefix="$(arg prefix)"
     eth_device="$(arg eth_device)"
-    joint1_mechanical_reduction="$(arg joint1_mechanical_reduction)"
-    joint2_mechanical_reduction="$(arg joint2_mechanical_reduction)"
-    joint3_mechanical_reduction="$(arg joint3_mechanical_reduction)"
-    joint4_mechanical_reduction="$(arg joint4_mechanical_reduction)"
-    joint5_mechanical_reduction="$(arg joint5_mechanical_reduction)"
-    joint6_mechanical_reduction="$(arg joint6_mechanical_reduction)"
-    joint7_mechanical_reduction="$(arg joint7_mechanical_reduction)"/>
+    yaw1_mechanical_reduction="$(arg yaw1_mechanical_reduction)"
+    yaw2_mechanical_reduction="$(arg yaw2_mechanical_reduction)"
+    elev1_j1_mechanical_reduction="$(arg elev1_j1_mechanical_reduction)"
+    elev1_j2_mechanical_reduction="$(arg elev1_j2_mechanical_reduction)"
+    wrist_yaw_mechanical_reduction="$(arg wrist_yaw_mechanical_reduction)"
+    wrist_pitch_mechanical_reduction="$(arg wrist_pitch_mechanical_reduction)"
+    wrist_roll_mechanical_reduction="$(arg wrist_roll_mechanical_reduction)"/>
 </robot>

Commit message: Update joint ordering; streamline logic in HAND_GUIDED mode (#49)
* Debug wrist yaw brake lockup

* Update joint ordering to match ecat ordering

* Debug joint order

File: description/ros2_control/seven_dof.ros2_control.xacro (robot description, xacro)
@@ -65,16 +65,4 @@
         <state_interface name="hand_guided"/>
       </joint>
-      <joint name="${prefix}wrist_yaw">
-        <command_interface name="position"/>
-        <command_interface name="velocity"/>
-        <command_interface name="hand_guided"/>
-        <command_interface name="quick_stop"/>
-        <command_interface name="compensate_for_removed_load"/>
-        <command_interface name="compensate_for_added_load"/>
-        <state_interface name="position"/>
-        <state_interface name="velocity"/>
-        <state_interface name="acceleration"/>
-        <state_interface name="hand_guided"/>
-      </joint>
       <joint name="${prefix}wrist_pitch">
         <command_interface name="position"/>
@@ -90,4 +78,16 @@
       </joint>
       <joint name="${prefix}wrist_roll">
+        <command_interface name="position"/>
+        <command_interface name="velocity"/>
+        <command_interface name="hand_guided"/>
+        <command_interface name="quick_stop"/>
+        <command_interface name="compensate_for_removed_load"/>
+        <command_interface name="compensate_for_added_load"/>
+        <state_interface name="position"/>
+        <state_interface name="velocity"/>
+        <state_interface name="acceleration"/>
+        <state_interface name="hand_guided"/>
+      </joint>
+      <joint name="${prefix}wrist_yaw">
         <command_interface name="position"/>
         <command_interface name="velocity"/>
