Commit message: new readme, documentation, 1dof version, images

File: description/urdf/two_dof_macro.urdf.xacro (robot description, xacro)
@@ -3,10 +3,10 @@
   <xacro:macro name="two_dof" params="parent prefix *origin">
   <!-- Constants for robot dimensions -->
-  <xacro:property name="mass" value="1" /> <!-- arbitrary value for mass -->
-  <xacro:property name="width" value="0.1" /> <!-- Square dimensions (widthxwidth) of beams -->
-  <xacro:property name="height1" value="2" /> <!-- Link 1 -->
-  <xacro:property name="height2" value="1" /> <!-- Link 2 -->
-  <xacro:property name="height3" value="1" /> <!-- Link 3 -->
-  <xacro:property name="axel_offset" value="0.05" /> <!-- Space btw top of beam and the each joint -->
+  <xacro:property name="mass" value="1" />
+  <xacro:property name="width" value="0.1" />
+  <xacro:property name="height1" value="2" />
+  <xacro:property name="height2" value="1" />
+  <xacro:property name="height3" value="1" />
+  <xacro:property name="axel_offset" value="0.00" />
   <joint name="${prefix}base_joint" type="fixed">
     <xacro:insert_block name="origin" />
@@ -16,31 +16,22 @@
   <!-- Base Link -->
   <link name="${prefix}base_link">
-    <collision>
-      <origin xyz="0 0 ${height1/2}" rpy="0 0 0"/>
-      <geometry>
-        <box size="${width} ${width} ${height1}"/>
-      </geometry>
-    </collision>
-    <visual>
-      <origin xyz="0 0 ${height1/2}" rpy="0 0 0"/>
-      <geometry>
-        <box size="${width} ${width} ${height1}"/>
-      </geometry>
-      <material name="orange"/>
-    </visual>
-    <inertial>
-      <origin xyz="0 0 ${height1/2}" rpy="0 0 0"/>
-      <mass value="${mass}"/>
-      <inertia
-        ixx="${mass / 12.0 * (width*width + height1*height1)}" ixy="0.0" ixz="0.0"
-        iyy="${mass / 12.0 * (height1*height1 + width*width)}" iyz="0.0"
-        izz="${mass / 12.0 * (width*width + width*width)}"/>
-    </inertial>
-  </link>
+      <visual>
+        <origin xyz="0 0 0" rpy="0 0 0"/>
+        <geometry>
+          <mesh filename="package://synapticon_ros2_control/meshes/flywheel.stl" scale="0.005 0.005 0.005"/>
+        </geometry>
+      </visual>
+      <collision>
+        <origin xyz="0 0 0" rpy="0 0 0"/>
+        <geometry>
+          <mesh filename="package://synapticon_ros2_control/meshes/flywheel.stl" scale="0.005 0.005 0.005"/>
+        </geometry>
+      </collision>
+   </link>
   <joint name="${prefix}joint1" type="continuous">
     <parent link="${prefix}base_link"/>
     <child link="${prefix}link1"/>
-    <origin xyz="0 ${width} ${height1 - axel_offset}" rpy="0 0 0"/>
-    <axis xyz="0 1 0"/>
+    <origin xyz="0 0 0" rpy="0 0 0"/>
+    <axis xyz="0 0 1"/>
     <dynamics damping="0.7"/>
     <limit effort="100" velocity="1.0"/>
@@ -48,58 +39,60 @@
   <!-- Middle Link -->
   <link name="${prefix}link1">
-    <collision>
-      <origin xyz="0 0 ${height2/2 - axel_offset}" rpy="0 0 0"/>
-      <geometry>
-        <box size="${width} ${width} ${height2}"/>
-      </geometry>
-    </collision>
-    <visual>
-      <origin xyz="0 0 ${height2/2 - axel_offset}" rpy="0 0 0"/>
-      <geometry>
-        <box size="${width} ${width} ${height2}"/>
-      </geometry>
-      <material name="yellow"/>
-    </visual>
-    <inertial>
-      <origin xyz="0 0 ${height2/2 - axel_offset}" rpy="0 0 0"/>
-      <mass value="${mass}"/>
-      <inertia
-        ixx="${mass / 12.0 * (width*width + height2*height2)}" ixy="0.0" ixz="0.0"
-        iyy="${mass / 12.0 * (height2*height2 + width*width)}" iyz="0.0"
-        izz="${mass / 12.0 * (width*width + width*width)}"/>
-    </inertial>
-  </link>
-  <joint name="${prefix}joint2" type="continuous">
+      <visual>
+        <origin xyz="0 0 0" rpy="0 0 0"/>
+        <geometry>
+          <mesh filename="package://synapticon_ros2_control/meshes/motor.stl" scale="0.005 0.005 0.005"/>
+        </geometry>
+      </visual>
+      <collision>
+        <origin xyz="0 0 0" rpy="0 0 0"/>
+        <geometry>
+          <mesh filename="package://synapticon_ros2_control/meshes/motor.stl" scale="0.005 0.005 0.005"/>
+        </geometry>
+      </collision>
+    </link>
+  <joint name="${prefix}fixed_joint" type="fixed">  <!-- Renamed to avoid duplicate base_joint -->
     <parent link="${prefix}link1"/>
     <child link="${prefix}link2"/>
-    <origin xyz="0 ${width} ${height2 - axel_offset*2}" rpy="0 0 0"/>
-    <axis xyz="0 1 0"/>
+    <origin xyz="0 1.1 0" rpy="0 0 0"/>
+  </joint>
+  <!-- Fixed Link -->
+  <link name="${prefix}link2">
+      <visual>
+        <origin xyz="0 0 0" rpy="0 0 0"/>
+        <geometry>
+          <mesh filename="package://synapticon_ros2_control/meshes/motor.stl" scale="0.005 0.005 0.005"/>
+        </geometry>
+      </visual>
+      <collision>
+        <origin xyz="0 0 0" rpy="0 0 0"/>
+        <geometry>
+          <mesh filename="package://synapticon_ros2_control/meshes/motor.stl" scale="0.005 0.005 0.005"/>
+        </geometry>
+      </collision>
+   </link>
+  <joint name="${prefix}joint2" type="continuous">
+    <parent link="${prefix}link2"/>
+    <child link="${prefix}link3"/>
+    <origin xyz="0 0 0" rpy="0 0 0"/>
+    <axis xyz="0 0 1"/>
     <dynamics damping="0.7"/>
     <limit effort="100" velocity="1.0"/>
   </joint>
-  <!-- Top Link -->
-  <link name="${prefix}link2">
-    <collision>
-      <origin xyz="0 0 ${height3/2 - axel_offset}" rpy="0 0 0"/>
-      <geometry>
-        <box size="${width} ${width} ${height3}"/>
-      </geometry>
-    </collision>
-    <visual>
-      <origin xyz="0 0 ${height3/2 - axel_offset}" rpy="0 0 0"/>
-      <geometry>
-        <box size="${width} ${width} ${height3}"/>
-      </geometry>
-      <material name="orange"/>
-    </visual>
-    <inertial>
-      <origin xyz="0 0 ${height3/2 - axel_offset}" rpy="0 0 0"/>
-      <mass value="${mass}"/>
-      <inertia
-        ixx="${mass / 12.0 * (width*width + height3*height3)}" ixy="0.0" ixz="0.0"
-        iyy="${mass / 12.0 * (height3*height3 + width*width)}" iyz="0.0"
-        izz="${mass / 12.0 * (width*width + width*width)}"/>
-    </inertial>
-  </link>
+  <!-- Flywheel 2 Link -->
+  <link name="${prefix}link3">
+      <visual>
+        <origin xyz="0 0 0" rpy="0 0 0"/>
+        <geometry>
+          <mesh filename="package://synapticon_ros2_control/meshes/flywheel.stl" scale="0.005 0.005 0.005"/>
+        </geometry>
+      </visual>
+      <collision>
+        <origin xyz="0 0 0" rpy="0 0 0"/>
+        <geometry>
+          <mesh filename="package://synapticon_ros2_control/meshes/flywheel.stl" scale="0.005 0.005 0.005"/>
+        </geometry>
+      </collision>
+   </link>
   </xacro:macro>
 </robot>
